File: quadrotor.sch (EAGLE design)
At the start: 10 parts, among them X1 16MHZ

Commit message: done bluetooth protocal
Parts:
- added C4: 0.1uF, eagle-ltspice:CC0603
- added C7, C8: 1uF, eagle-ltspice:CC0603
- added JP2, JP3, JP4: (no value), pinhead:PINHD-1X2
- added JP5: (no value), pinhead:PINHD-1X6/90
- added JP8: (no value), pinhead:PINHD-1X6
- added JP9: (no value), pinhead:PINHD-1X2/90
- added R1, R2: 100k, eagle-ltspice:RR0603
- added S1: DTSM-3, switch-tact:DTSM-3
- added U$1: RT9013, quadrotor:RT9013
- C1, C2: value (none) -> 22pF
- C3: value (none) -> 0.1uF
- T1, T2, T3, T4: value (none) -> AO3400; device zetex:PMOSSOT23 -> zetex:NMOSSOT23
- X1: device IQD-Frequency-Products:CRYSTALS-NOGND-HC49 -> IQD-Frequency-Products:CRYSTALS-NOGND-12SMX-A
Connections:
- net N$3 renamed AREF
- new net ADC6: ATMEGA328P.ADC6
- new net ADC7: ATMEGA328P.ADC7
- new net MISO: ATMEGA328P.PB4(MISO), JP5.3
- new net MOSI: ATMEGA328P.PB3(MOSI/OC2), JP5.4
- new net N$10: JP3.1, T3.D
- new net N$4: JP1.1, T1.D
- new net N$6: JP2.1, T2.D
- new net N$9: JP4.1, T4.D
- new net PB0: ATMEGA328P.PB0(ICP)
- new net PC0: ATMEGA328P.PC0(ADC0)
- new net PC1: ATMEGA328P.PC1(ADC1)
- new net PC2: ATMEGA328P.PC2(ADC2)
- new net PC3: ATMEGA328P.PC3(ADC3)
- new net PC4: ATMEGA328P.PC4(ADC4/SDA)
- new net PC5: ATMEGA328P.PC5(ADC5/SCL)
- new net PD0: ATMEGA328P.PD0(RXD), JP8.4
- new net PD1: ATMEGA328P.PD1(TXD), JP8.5
- new net PD2: ATMEGA328P.PD2(INT0), JP8.6
- new net PD3: ATMEGA328P.PD3(INT1)
- new net PD4: ATMEGA328P.PD4(XCK/T0)
- new net PD7: ATMEGA328P.PD7(AIN1)
- new net RESET: ATMEGA328P.PC6(/RESET), JP5.1, R2.1, S1.2
- new net SCK: ATMEGA328P.PB5(SCK), JP5.2
- new net VIN: C7.1, JP1.2, JP2.2, JP3.2, JP4.2, JP5.6, JP9.1, R1.2, U$1.EN, U$1.VIN
- net GND: now also C4.2, C7.2, C8.2, JP5.5, JP8.3, JP9.2, R1.1, S1.1, T1.S, T2.S, T3.S, T4.S, U$1.GND
- net N$1: now also C2.2; no longer C1.2
- net N$2: now also C1.2; no longer C2.2
- net VCC: now also ATMEGA328P.AVCC, C4.1, C8.1, JP8.1, JP8.2, R2.2, U$1.VOUT
Other:
- moved on the sheet: C1, C2, C3, JP1, T3, T4

Commit message: mostly done layout and is routing now
Parts:
- removed C1, C2: 22pF, eagle-ltspice:CC0603
- removed JP8: (no value), pinhead:PINHD-1X6
- added C10, C11, C12, C13, C14, C15, C16, C17, C18, C5, C6, C9: 0.1uF, eagle-ltspice:CC0603
- added JP6: (no value), pinhead:PINHD-1X4
- added LED1: POWER, eagle-ltspice:LED_ESML0603
- added R3: 470, eagle-ltspice:RR0603
- added SW1: (no value), special:SW_DIP-5
- added U$2: BLT-HC05, quadrotor:BLT-HC05
- added U$3, U$4, U$5, U$6: 720-MSHELL, quadrotor:720-MSHELL
- JP5: device pinhead:PINHD-1X6/90 -> pinhead:PINHD-1X6
- JP9: device pinhead:PINHD-1X2/90 -> pinhead:PINHD-1X2
- X1: device IQD-Frequency-Products:CRYSTALS-NOGND-12SMX-A -> murata-filter:CSTCR6M00G53Z
Connections:
- removed net PD0: ATMEGA328P.PD0(RXD), JP8.4
- removed net PD1: ATMEGA328P.PD1(TXD), JP8.5
- new net N$11: SW1.8, U$2.VCC
- new net N$12: SW1.7, U$2.TX
- new net N$13: SW1.6, U$2.RX
- new net N$14: JP9.1, SW1.1
- new net N$15: C12.2, C17.1, U$4.SHELL
- new net N$16: C13.2, C16.1, U$6.SHELL
- new net N$3: C14.2, C15.1, U$5.SHELL
- new net N$5: C11.2, C18.1, U$3.SHELL
- new net N$7: SW1.9, U$2.EN
- new net N$8: LED1.A, R3.1
- new net PD0/RX: ATMEGA328P.PD0(RXD), JP6.3, SW1.4
- new net PD1/TX: ATMEGA328P.PD1(TXD), JP6.2, SW1.5
- net GND: now also C11.1, C12.1, C13.1, C14.1, JP5.6, JP6.4, LED1.C, U$2.GND, X1.2; no longer C1.1, C2.1, JP5.5, JP8.3
- net MISO: now also JP5.4; no longer JP5.3
- net MOSI: now also JP5.5; no longer JP5.4
- net N$1: no longer C2.2
- net N$10: now also C9.1
- net N$2: now also X1.3; no longer C1.2, X1.2
- net N$4: now also C5.1
- net N$6: now also C6.1
- net N$9: now also C10.1
- net PD2: now also U$2.STATE; no longer JP8.6
- net RESET: now also JP5.2; no longer JP5.1
- net SCK: now also JP5.3; no longer JP5.2
- net VCC: now also SW1.2, SW1.3; no longer JP8.1, JP8.2
- net VIN: now also C10.2, C15.2, C16.2, C17.2, C18.2, C5.2, C6.2, C9.2, JP5.1, JP6.1, R3.2, SW1.10; no longer JP5.6, JP9.1
Other:
- moved on the sheet: ATMEGA328P, C3, C4, C7, C8, JP1, JP2, JP3, JP4, JP5, JP9, R1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

Commit message: basically done pcb layout
Parts:
- added U$7: MPU-6050, quadrotor:MPU-6050
Connections:
- net GND: now also U$7.GND
- net PC4: now also U$7.SDA
- net PC5: now also U$7.SCL
- net PD3: now also U$7.INT
- net VCC: now also R3.2, U$7.VCC
- net VIN: no longer R3.2
Other:
- moved on the sheet: JP5
Changed lines of the file:
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@@
 <part name="U$6" library="quadrotor" deviceset="720-MSHELL" device=""/>
 <part name="SW1" library="special" deviceset="SW_DIP-5" device=""/>
+<part name="U$7" library="quadrotor" deviceset="MPU-6050" device=""/>
 </parts>
 <sheets>
@@
 <instance part="S1" gate="G$1" x="10.16" y="76.2" rot="R270"/>
 <instance part="SUPPLY2" gate="G$1" x="43.18" y="114.3"/>
-<instance part="JP5" gate="A" x="149.86" y="116.84"/>
+<instance part="JP5" gate="A" x="157.48" y="111.76"/>
 <instance part="JP9" gate="G$1" x="177.8" y="116.84" rot="MR0"/>
 <instance part="R3" gate="G$1" x="236.22" y="30.48" rot="R90"/>
@@
 <instance part="U$6" gate="M" x="210.82" y="20.32"/>
 <instance part="SW1" gate="A" x="213.36" y="114.3" rot="R180"/>
+<instance part="U$7" gate="U" x="269.24" y="119.38"/>
 </instances>
 <busses>
@@
 <segment>
 <pinref part="JP5" gate="A" pin="6"/>
-<wire x1="147.32" y1="111.76" x2="134.62" y2="111.76" width="0.1524" layer="91"/>
-<label x="134.62" y="111.76" size="1.778" layer="95"/>
+<wire x1="154.94" y1="106.68" x2="142.24" y2="106.68" width="0.1524" layer="91"/>
+<label x="142.24" y="106.68" size="1.778" layer="95"/>
+</segment>
+<segment>
+<pinref part="U$7" gate="U" pin="GND"/>
+<wire x1="269.24" y1="116.84" x2="261.62" y2="116.84" width="0.1524" layer="91"/>
+<label x="261.62" y="116.84" size="1.778" layer="95"/>
 </segment>
 </net>
@@
 <pinref part="SW1" gate="A" pin="2"/>
 <pinref part="SW1" gate="A" pin="3"/>
+</segment>
+<segment>
+<pinref part="U$7" gate="U" pin="VCC"/>
+<wire x1="269.24" y1="119.38" x2="261.62" y2="119.38" width="0.1524" layer="91"/>
+<label x="261.62" y="119.38" size="1.778" layer="95"/>
+</segment>
+<segment>
+<pinref part="R3" gate="G$1" pin="2"/>
+<wire x1="236.22" y1="35.56" x2="236.22" y2="40.64" width="0.1524" layer="91"/>
+<label x="238.76" y="40.64" size="1.778" layer="95"/>
+<wire x1="236.22" y1="40.64" x2="243.84" y2="40.64" width="0.1524" layer="91"/>
 </segment>
 </net>
@@
 </segment>
 <segment>
-<pinref part="R3" gate="G$1" pin="2"/>
-<wire x1="236.22" y1="35.56" x2="236.22" y2="40.64" width="0.1524" layer="91"/>
-<label x="238.76" y="40.64" size="1.778" layer="95"/>
-<wire x1="236.22" y1="40.64" x2="243.84" y2="40.64" width="0.1524" layer="91"/>
-</segment>
-<segment>
 <label x="223.52" y="119.38" size="1.778" layer="95"/>
 <pinref part="SW1" gate="A" pin="10"/>
@@
 <segment>
 <pinref part="JP5" gate="A" pin="1"/>
-<wire x1="147.32" y1="124.46" x2="134.62" y2="124.46" width="0.1524" layer="91"/>
-<label x="134.62" y="124.46" size="1.778" layer="95"/>
+<wire x1="154.94" y1="119.38" x2="142.24" y2="119.38" width="0.1524" layer="91"/>
+<label x="142.24" y="119.38" size="1.778" layer="95"/>
 </segment>
 </net>
@@
 <label x="91.44" y="66.04" size="1.778" layer="95"/>
 </segment>
+<segment>
+<pinref part="U$7" gate="U" pin="SDA"/>
+<wire x1="269.24" y1="111.76" x2="261.62" y2="111.76" width="0.1524" layer="91"/>
+<label x="261.62" y="111.76" size="1.778" layer="95"/>
+</segment>
 </net>
 <net name="PC5" class="0">
@@
 <label x="91.44" y="63.5" size="1.778" layer="95"/>
 </segment>
+<segment>
+<pinref part="U$7" gate="U" pin="SCL"/>
+<wire x1="269.24" y1="114.3" x2="261.62" y2="114.3" width="0.1524" layer="91"/>
+<label x="261.62" y="114.3" size="1.778" layer="95"/>
+</segment>
 </net>
 <net name="ADC6" class="0">
@@
 <label x="91.44" y="45.72" size="1.778" layer="95"/>
 </segment>
+<segment>
+<pinref part="U$7" gate="U" pin="INT"/>
+<wire x1="294.64" y1="111.76" x2="302.26" y2="111.76" width="0.1524" layer="91"/>
+<label x="297.18" y="111.76" size="1.778" layer="95"/>
+</segment>
 </net>
 <net name="PD4" class="0">
@@
 </segment>
 <segment>
-<wire x1="134.62" y1="114.3" x2="147.32" y2="114.3" width="0.1524" layer="91"/>
+<wire x1="142.24" y1="109.22" x2="154.94" y2="109.22" width="0.1524" layer="91"/>
 <pinref part="JP5" gate="A" pin="5"/>
-<label x="134.62" y="114.3" size="1.778" layer="95"/>
-<label x="134.62" y="114.3" size="1.778" layer="95"/>
+<label x="142.24" y="109.22" size="1.778" layer="95"/>
+<label x="142.24" y="109.22" size="1.778" layer="95"/>
 </segment>
 </net>
@@
 </segment>
 <segment>
-<wire x1="134.62" y1="116.84" x2="147.32" y2="116.84" width="0.1524" layer="91"/>
-<label x="134.62" y="116.84" size="1.778" layer="95"/>
+<wire x1="142.24" y1="111.76" x2="154.94" y2="111.76" width="0.1524" layer="91"/>
+<label x="142.24" y="111.76" size="1.778" layer="95"/>
 <pinref part="JP5" gate="A" pin="4"/>
 </segment>
@@
 </segment>
 <segment>
-<wire x1="134.62" y1="119.38" x2="147.32" y2="119.38" width="0.1524" layer="91"/>
-<label x="134.62" y="119.38" size="1.778" layer="95"/>
+<wire x1="142.24" y1="114.3" x2="154.94" y2="114.3" width="0.1524" layer="91"/>
+<label x="142.24" y="114.3" size="1.778" layer="95"/>
 <pinref part="JP5" gate="A" pin="3"/>
 </segment>
@@
 </segment>
 <segment>
-<wire x1="134.62" y1="121.92" x2="147.32" y2="121.92" width="0.1524" layer="91"/>
+<wire x1="142.24" y1="116.84" x2="154.94" y2="116.84" width="0.1524" layer="91"/>
 <pinref part="JP5" gate="A" pin="2"/>
-<label x="134.62" y="121.92" size="1.778" layer="95"/>
-</segment>
-</net>
+<label x="142.24" y="116.84" size="1.778" layer="95"/>
+</segment>
+</net>

Commit message: basically done v1 brd
Parts:
- renumbered LED1 to POW
Changed lines of the file:
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@@
 <part name="JP9" library="pinhead" deviceset="PINHD-1X2" device=""/>
 <part name="R3" library="eagle-ltspice" deviceset="R" device="R0603" value="470"/>
-<part name="LED1" library="eagle-ltspice" deviceset="LED_E" device="SML0603" value="POWER"/>
+<part name="POW" library="eagle-ltspice" deviceset="LED_E" device="SML0603" value="POWER"/>
 <part name="GND11" library="supply1" deviceset="GND" device=""/>
 <part name="GND12" library="supply1" deviceset="GND" device=""/>
@@
 <part name="C17" library="eagle-ltspice" deviceset="C" device="C0603" value="0.1uF"/>
 <part name="C18" library="eagle-ltspice" deviceset="C" device="C0603" value="0.1uF"/>
-<part name="U$3" library="quadrotor" deviceset="720-MSHELL" device=""/>
 <part name="U$4" library="quadrotor" deviceset="720-MSHELL" device=""/>
 <part name="U$5" library="quadrotor" deviceset="720-MSHELL" device=""/>
@@
 <part name="SW1" library="special" deviceset="SW_DIP-5" device=""/>
 <part name="U$7" library="quadrotor" deviceset="MPU-6050" device=""/>
+<part name="U$3" library="quadrotor" deviceset="720-MSHELL" device=""/>
 </parts>
 <sheets>
@@
 <instance part="JP9" gate="G$1" x="177.8" y="116.84" rot="MR0"/>
 <instance part="R3" gate="G$1" x="236.22" y="30.48" rot="R90"/>
-<instance part="LED1" gate="G$1" x="236.22" y="20.32"/>
+<instance part="POW" gate="G$1" x="236.22" y="20.32"/>
 <instance part="GND11" gate="1" x="236.22" y="7.62"/>
 <instance part="GND12" gate="1" x="231.14" y="99.06"/>
@@
 <instance part="C17" gate="G$1" x="210.82" y="81.28" rot="R180"/>
 <instance part="C18" gate="G$1" x="154.94" y="81.28" rot="R180"/>
-<instance part="U$3" gate="M" x="154.94" y="76.2"/>
 <instance part="U$4" gate="M" x="210.82" y="76.2"/>
 <instance part="U$5" gate="M" x="154.94" y="20.32"/>
@@
 <instance part="SW1" gate="A" x="213.36" y="114.3" rot="R180"/>
 <instance part="U$7" gate="U" x="269.24" y="119.38"/>
+<instance part="U$3" gate="M" x="154.94" y="76.2"/>
 </instances>
 <busses>
@@
 </segment>
 <segment>
-<pinref part="LED1" gate="G$1" pin="C"/>
+<pinref part="POW" gate="G$1" pin="C"/>
 <wire x1="236.22" y1="15.24" x2="236.22" y2="10.16" width="0.1524" layer="91"/>
 <pinref part="GND11" gate="1" pin="GND"/>
@@
 <segment>
 <pinref part="R3" gate="G$1" pin="1"/>
-<pinref part="LED1" gate="G$1" pin="A"/>
+<pinref part="POW" gate="G$1" pin="A"/>
 <wire x1="236.22" y1="25.4" x2="236.22" y2="22.86" width="0.1524" layer="91"/>
 </segment>
